File: dboard/dboard.kicad_pcb (KiCad board)
At the start: 2 copper layers, 49 x 11 mm, 10 parts, among them J1 Conn_01x04, U1 SRV05-4

Commit message: first
Parts:
- removed R3: 1M, Resistor_SMD:R_1206_3216Metric
- added C2: 1u, Capacitor_SMD:C_0402_1005Metric, B.Cu at (-9.77, 2.53)
- added C3: 100n, Capacitor_SMD:C_0402_1005Metric, B.Cu at (-11.1, 8.37)
- added C4: 4.7u, Capacitor_SMD:C_0402_1005Metric, B.Cu at (-12.1, 8.37)
- added D1: D_TVS, other:BSD3C051V, B.Cu at (-8.25, 6.38)
- added L1: L_Ferrite, other:BEADC1005X55N, B.Cu at (-9.94, 9.31)
- added L2: L_Ferrite, other:BEADC1005X55N, B.Cu at (-8.71, 8.37)
- added L3: L_Ferrite, other:BEADC1005X55N, B.Cu at (-9.30, 4.70)
- added U2: XC6206P332MR, Package_TO_SOT_SMD:SOT-23, B.Cu at (-12.1, 3.43)
- C1: value 470n -> 1u; footprint Capacitor_SMD:C_0805_2012Metric -> Capacitor_SMD:C_0402_1005Metric
- R1, R2: footprint Resistor_SMD:R_0603_1608Metric -> Resistor_SMD:R_0402_1005Metric
- U1: value SRV05-4 -> TPD2E2U06DRLR; footprint Package_TO_SOT_SMD:SOT-23-6 -> other:SOTFL50P160X60-5N
- moved H1 42.0 mm to (21.0, 5.50)
- moved H2 38.0 mm to (-21.0, 5.50)
- moved J1 27.7 mm to (14.1, 7.42)
- moved C1 20.9 mm to (-12.1, 6.44)
- moved U1 16.8 mm to (9.03, 5.85), turned to -90 degrees
- moved F1 5.59 mm to (-14.0, 7.83)
- moved R1 5.33 mm to (6.24, 2.93)
- moved R2 5.15 mm to (7.27, 2.93)
Connections:
- C1 pad 1: SHIELD -> +5V
- F1 pad 2: VBUS -> Net-(C3-Pad1)
- J1 pad 1: +5V -> +3V3
- J1 pad 2: D+ -> GND
- J1 pad 3: D- -> D+
- J1 pad 4: GND -> D-
- U1 pad 1: (no net) -> D+
- U1 pad 2: GND -> D+
- U1 pad 4: D+ -> GND
- U1 pad 5: +5V -> D+
- USB1 pad 1: GND -> USBGND
- USB1 pad 12: GND -> USBGND
- USB1 pad 3: (no net) -> unconnected-(USB1-Pad3)
- USB1 pad 9: (no net) -> unconnected-(USB1-Pad9)
Routing:
- net +3V3: track 0.00 -> 30.2 mm, vias 0 -> 2
- net GND: track 40.3 -> 61.1 mm, vias 7 -> 1
- net USBGND: track 0.00 -> 16.5 mm, vias 0 -> 2
- net SHIELD: track 74.6 -> 82.2 mm, vias 0 -> 1
- net D+: track 29.5 -> 24.1 mm
- net D-: track 27.6 -> 22.9 mm
- net +5V: track 7.74 -> 3.64 mm
- net Net-(C3-Pad1): track 0.00 -> 3.57 mm
- net Net-(R1-Pad2): track 12.5 -> 10.6 mm
- net Net-(R2-Pad2): track 7.41 -> 8.71 mm, vias 0 -> 2
- net VBUS: track 18.8 -> 17.7 mm, vias 3 -> 2
Other:
- board size 49 x 11 mm -> 53 x 11 mm
- net class Default removed
- net class Power removed
