File: dboard/dboard.kicad_pcb (KiCad board)
At the start: 2 copper layers, 53 x 11 mm, 18 parts, among them J1 Conn_01x04, U1 TPD2E2U06DRLR, U2 XC6206P332MR

Commit message: rearranged
Parts:
- moved U1 1.33 mm to (7.50, 7.56)
- moved L3 1.15 mm to (-8.15, 4.72)
- moved U2 0.92 mm to (-12.7, 2.72), turned to 180 degrees
- moved D1 0.90 mm to (-7.35, 6.32)
- moved R2 0.64 mm to (6.63, 2.89)
- moved R1 0.62 mm to (5.62, 2.88)
- moved C2 0.52 mm to (-10.2, 2.81), turned to 90 degrees
- moved L2 0.12 mm to (-8.59, 8.37)
- moved L1 0.12 mm to (-9.82, 9.31)
Connections:
- L2 pad 1: USBGND -> GND
- USB1 pad 1: USBGND -> GND
- USB1 pad 12: USBGND -> GND
Routing:
- net USBGND: track 16.5 -> 0.00 mm, vias 2 -> 0
- net +5V: track 3.64 -> 5.82 mm
- net Net-(R2-Pad2): track 8.71 -> 8.13 mm
- net D+: track 23.9 -> 23.3 mm
- net GND: track 59.9 -> 60.4 mm, vias 2 -> 4

Commit message: curvy
Parts:
- moved D1 1.76 mm to (-6.16, 5.03), turned to 90 degrees
- moved U2 1.62 mm to (-11.1, 2.67)
- moved C2 1.58 mm to (-8.64, 2.67)
- moved L3 0.60 mm to (-7.74, 5.16), turned to -90 degrees
- moved L2 0.27 mm to (-8.86, 8.36)
- moved L1 0.20 mm to (-10.0, 9.29)
- renumbered USB1 to J1, J1 to J2
Routing:
- net D-: track 22.7 -> 19.8 mm
- net SHIELD: track 82.1 -> 80.1 mm
- net VBUS: track 17.7 -> 16.1 mm
- net +3V3: track 32.9 -> 31.4 mm
- net GND: track 60.4 -> 61.2 mm
- net +5V: track 5.82 -> 6.52 mm
- net D+: track 23.3 -> 22.8 mm

Commit message: changes
Parts:
- moved D2 24.7 mm to (-10.5, 6.25), turned to 180 degrees
- moved C1 1.82 mm to (-11.6, 4.73), turned to 0 degrees
Connections:
- D2 pad 2: +3V3 -> +5V
Routing:
- net SHIELD: track 80.1 -> 87.1 mm
- net GND: track 61.2 -> 65.9 mm
- net +3V3: track 31.4 -> 28.8 mm
Other:
- board text added: "v0.1"
